File: hardware/waveform.kicad_pcb (KiCad board)
At the start: 2 copper layers, 229 x 231 mm, 190 parts, among them J1 PHASE_POLARITY, J2 PHASE_POLARITY, J3 PHASE_POLARITY, J4 PHASE_POLARITY, J5 POWER_12V, J6 WAVE_OUT, U1 NE555P, U10 TL082CP, U11 TL082CP, U12 TL082CP, U13 TL082CP, U14 TL082CP, U15 TL082CP, U16 TL082CP, U2 CD4013BE, U3 TL082CP, U4 TL082CP, U5 TL082CP, U6 TL082CP, U7 TL082CP, U8 TL082CP, U9 TL082CP

Commit message: Redraw waveform schematic as wired functional blocks for readable EDA import
Split TL082 amplifier and power units, replace the component grid with a single wired schematic and local net labels, and update both KiCad and EAGLE exchanges. Preserve all PCB copper and pad geometry; verify 491 pin connections, zero ERC/DRC issues, and EAGLE PCB round-trip checks. Add clearly named RevB wired download packages.
Connections:
- net AC_SQUARE renamed /AC_SQUARE
- net CLOCK_2K renamed /CLOCK_2K
- net CTRL renamed /CTRL
- net DIGITAL_1K renamed /DIGITAL_1K
- net DISCHARGE renamed /DISCHARGE
- net D_FEEDBACK renamed /D_FEEDBACK
- net FREQ_R renamed /FREQ_R
- net GND renamed /GND
- net H1_AMPLITUDE renamed /H1_AMPLITUDE
- net H1_AP1 renamed /H1_AP1
- net H1_AP2 renamed /H1_AP2
- net H1_APINV1 renamed /H1_APINV1
- net H1_APINV2 renamed /H1_APINV2
- net H1_BPF1 renamed /H1_BPF1
- net H1_BPF2 renamed /H1_BPF2
- net H1_INV1 renamed /H1_INV1
- net H1_INV2 renamed /H1_INV2
- net H1_LP1 renamed /H1_LP1
- net H1_LP2 renamed /H1_LP2
- net H1_NEG renamed /H1_NEG
- net H1_NODE1 renamed /H1_NODE1
- net H1_NODE2 renamed /H1_NODE2
- net H1_OUT renamed /H1_OUT
- net H1_PHR1 renamed /H1_PHR1
- net H1_PHR2 renamed /H1_PHR2
- net H1_POLINV renamed /H1_POLINV
- net H1_SELECT renamed /H1_SELECT
- net H1_TUNE1 renamed /H1_TUNE1
- net H1_TUNE2 renamed /H1_TUNE2
- net H3_AMPLITUDE renamed /H3_AMPLITUDE
- net H3_AP1 renamed /H3_AP1
- net H3_AP2 renamed /H3_AP2
- net H3_APINV1 renamed /H3_APINV1
- net H3_APINV2 renamed /H3_APINV2
- net H3_BPF1 renamed /H3_BPF1
- net H3_BPF2 renamed /H3_BPF2
- net H3_INV1 renamed /H3_INV1
- net H3_INV2 renamed /H3_INV2
- net H3_LP1 renamed /H3_LP1
- net H3_LP2 renamed /H3_LP2
- net H3_NEG renamed /H3_NEG
- net H3_NODE1 renamed /H3_NODE1
- net H3_NODE2 renamed /H3_NODE2
- net H3_OUT renamed /H3_OUT
- net H3_PHR1 renamed /H3_PHR1
- net H3_PHR2 renamed /H3_PHR2
- net H3_POLINV renamed /H3_POLINV
- net H3_SELECT renamed /H3_SELECT
- net H3_TUNE1 renamed /H3_TUNE1
- net H3_TUNE2 renamed /H3_TUNE2
- net H5_AMPLITUDE renamed /H5_AMPLITUDE
- net H5_AP1 renamed /H5_AP1
- net H5_AP2 renamed /H5_AP2
- net H5_APINV1 renamed /H5_APINV1
- net H5_APINV2 renamed /H5_APINV2
- net H5_BPF1 renamed /H5_BPF1
- net H5_BPF2 renamed /H5_BPF2
- net H5_INV1 renamed /H5_INV1
- net H5_INV2 renamed /H5_INV2
- net H5_LP1 renamed /H5_LP1
- net H5_LP2 renamed /H5_LP2
- net H5_NEG renamed /H5_NEG
- net H5_NODE1 renamed /H5_NODE1
- net H5_NODE2 renamed /H5_NODE2
- net H5_OUT renamed /H5_OUT
- net H5_PHR1 renamed /H5_PHR1
- net H5_PHR2 renamed /H5_PHR2
- net H5_POLINV renamed /H5_POLINV
- net H5_SELECT renamed /H5_SELECT
- net H5_TUNE1 renamed /H5_TUNE1
- net H5_TUNE2 renamed /H5_TUNE2
- net H7_AMPLITUDE renamed /H7_AMPLITUDE
- net H7_AP1 renamed /H7_AP1
- net H7_AP2 renamed /H7_AP2
- net H7_APINV1 renamed /H7_APINV1
- net H7_APINV2 renamed /H7_APINV2
- net H7_BPF1 renamed /H7_BPF1
- net H7_BPF2 renamed /H7_BPF2
- net H7_INV1 renamed /H7_INV1
- net H7_INV2 renamed /H7_INV2
- net H7_LP1 renamed /H7_LP1
- net H7_LP2 renamed /H7_LP2
- net H7_NEG renamed /H7_NEG
- net H7_NODE1 renamed /H7_NODE1
- net H7_NODE2 renamed /H7_NODE2
- net H7_OUT renamed /H7_OUT
- net H7_PHR1 renamed /H7_PHR1
- net H7_PHR2 renamed /H7_PHR2
- net H7_POLINV renamed /H7_POLINV
- net H7_SELECT renamed /H7_SELECT
- net H7_TUNE1 renamed /H7_TUNE1
- net H7_TUNE2 renamed /H7_TUNE2
- net OUT renamed /OUT
- net RESTORE_INV renamed /RESTORE_INV
- net SOURCE_WIPER renamed /SOURCE_WIPER
- net SQ renamed /SQ
- net SQ_INV renamed /SQ_INV
- net SQ_INV_IN renamed /SQ_INV_IN
- net SUM_INV renamed /SUM_INV
- net SUM_NEG renamed /SUM_NEG
- net SUM_RAW renamed /SUM_RAW
- net TIMING renamed /TIMING
- net VCC renamed /VCC
- net VEE renamed /VEE
