File: hardware/waveform.kicad_sch (KiCad schematic)
At the start: 0 parts

Commit message: Redraw waveform schematic as wired functional blocks for readable EDA import
Split TL082 amplifier and power units, replace the component grid with a single wired schematic and local net labels, and update both KiCad and EAGLE exchanges. Preserve all PCB copper and pad geometry; verify 491 pin connections, zero ERC/DRC issues, and EAGLE PCB round-trip checks. Add clearly named RevB wired download packages.
Parts:
- added C1, C2, C4, C5, C6, C7, C8, C9: 10n, Waveform:C_Disc_D5.0mm_W2.5mm_P5.00mm, symbol Waveform:C
- added C10, C11, C12, C13, C14, C15: 3.3n, Waveform:C_Disc_D5.0mm_W2.5mm_P5.00mm, symbol Waveform:C
- added C16, C17, C18, C19, C20, C21: 2n, Waveform:C_Disc_D5.0mm_W2.5mm_P5.00mm, symbol Waveform:C
- added C22, C23, C24, C25, C26, C27: 1.5n, Waveform:C_Disc_D5.0mm_W2.5mm_P5.00mm, symbol Waveform:C
- added C28, C29: 47u/25V, Waveform:CP_Radial_D5.0mm_P2.00mm, symbol Waveform:CP
- added C3: 10u/25V, Waveform:CP_Radial_D5.0mm_P2.00mm, symbol Waveform:CP
- added C30, C31, C32, C33, C34, C35, C36, C37, C38, C39, C40, C41, C42, C43, C44, C45, C46, C47, C48, C49, C50, C51, C52, C53, C54, C55, C56, C57, C58, C59: 100n, Waveform:C_Disc_D5.0mm_W2.5mm_P5.00mm, symbol Waveform:C
- added J1, J2, J3, J4: PHASE_POLARITY, Waveform:PinHeader_1x03_P2.54mm_Vertical, symbol Waveform:CONN3
- added J5: POWER_12V, Waveform:PinHeader_1x03_P2.54mm_Vertical, symbol Waveform:CONN3
- added J6: WAVE_OUT, Waveform:PinHeader_1x02_P2.54mm_Vertical, symbol Waveform:CONN2
- added R1, R12, R13, R15, R16, R18, R19, R26, R27, R29, R30, R32, R33, R40, R41, R43, R44, R46, R47, R54, R55, R57, R58, R60, R61: 10k, Waveform:R_Axial_DIN0207_L6.3mm_D2.5mm_P7.62mm_Horizontal, symbol Waveform:R
- added R10, R21, R24, R35, R38, R49, R52, R7: 430, Waveform:R_Axial_DIN0207_L6.3mm_D2.5mm_P7.62mm_Horizontal, symbol Waveform:R
- added R11, R22, R25, R36, R39, R50, R53, R8: 470k, Waveform:R_Axial_DIN0207_L6.3mm_D2.5mm_P7.62mm_Horizontal, symbol Waveform:R
- added R14, R17, R28, R31, R42, R45, R56, R59, R69: 100, Waveform:R_Axial_DIN0207_L6.3mm_D2.5mm_P7.62mm_Horizontal, symbol Waveform:R
- added R2: 27k, Waveform:R_Axial_DIN0207_L6.3mm_D2.5mm_P7.62mm_Horizontal, symbol Waveform:R
- added R20, R23, R34, R37, R48, R51, R6, R9: 220k, Waveform:R_Axial_DIN0207_L6.3mm_D2.5mm_P7.62mm_Horizontal, symbol Waveform:R
- added R3: 1M, Waveform:R_Axial_DIN0207_L6.3mm_D2.5mm_P7.62mm_Horizontal, symbol Waveform:R
- added R4, R5, R62, R63, R64, R65, R66, R67, R68: 100k, Waveform:R_Axial_DIN0207_L6.3mm_D2.5mm_P7.62mm_Horizontal, symbol Waveform:R
- added RV1: 20k, Waveform:Potentiometer_Bourns_3296W_Vertical, symbol Waveform:POT
- added RV10, RV11, RV15, RV16, RV20, RV21, RV5, RV6: 200k, Waveform:Potentiometer_Bourns_3296W_Vertical, symbol Waveform:POT
- added RV12, RV17, RV22, RV7: 10k, Waveform:Potentiometer_Bourns_3296W_Vertical, symbol Waveform:POT
- added RV13, RV14, RV18, RV19, RV3, RV4, RV8, RV9: 200, Waveform:Potentiometer_Bourns_3296W_Vertical, symbol Waveform:POT
- added RV2: 100k, Waveform:Potentiometer_Bourns_3296W_Vertical, symbol Waveform:POT
- added TP1: CLOCK_2K, Waveform:TestPoint_THTPad_D1.5mm_Drill0.7mm, symbol Waveform:TP
- added TP10: H5_BPF2, Waveform:TestPoint_THTPad_D1.5mm_Drill0.7mm, symbol Waveform:TP
- added TP11: H5_AP2, Waveform:TestPoint_THTPad_D1.5mm_Drill0.7mm, symbol Waveform:TP
- added TP12: H5_OUT, Waveform:TestPoint_THTPad_D1.5mm_Drill0.7mm, symbol Waveform:TP
- added TP13: H7_BPF2, Waveform:TestPoint_THTPad_D1.5mm_Drill0.7mm, symbol Waveform:TP
- added TP14: H7_AP2, Waveform:TestPoint_THTPad_D1.5mm_Drill0.7mm, symbol Waveform:TP
- added TP15: H7_OUT, Waveform:TestPoint_THTPad_D1.5mm_Drill0.7mm, symbol Waveform:TP
- added TP16: SUM_RAW, Waveform:TestPoint_THTPad_D1.5mm_Drill0.7mm, symbol Waveform:TP
- added TP17: OUT, Waveform:TestPoint_THTPad_D1.5mm_Drill0.7mm, symbol Waveform:TP
- added TP18: GND, Waveform:TestPoint_THTPad_D1.5mm_Drill0.7mm, symbol Waveform:TP
- added TP2: SQ, Waveform:TestPoint_THTPad_D1.5mm_Drill0.7mm, symbol Waveform:TP
- added TP3: SQ_INV, Waveform:TestPoint_THTPad_D1.5mm_Drill0.7mm, symbol Waveform:TP
- added TP4: H1_BPF2, Waveform:TestPoint_THTPad_D1.5mm_Drill0.7mm, symbol Waveform:TP
- added TP5: H1_AP2, Waveform:TestPoint_THTPad_D1.5mm_Drill0.7mm, symbol Waveform:TP
- added TP6: H1_OUT, Waveform:TestPoint_THTPad_D1.5mm_Drill0.7mm, symbol Waveform:TP
- added TP7: H3_BPF2, Waveform:TestPoint_THTPad_D1.5mm_Drill0.7mm, symbol Waveform:TP
- added TP8: H3_AP2, Waveform:TestPoint_THTPad_D1.5mm_Drill0.7mm, symbol Waveform:TP
- added TP9: H3_OUT, Waveform:TestPoint_THTPad_D1.5mm_Drill0.7mm, symbol Waveform:TP
- added U1: NE555P, Waveform:DIP-8_W7.62mm, symbol Waveform:NE555
- added U10, U11, U12, U13, U14, U15, U16, U3, U4, U5, U6, U7, U8, U9: TL082CP, Waveform:DIP-8_W7.62mm, symbol Waveform:TL082
- added U2: CD4013BE, Waveform:DIP-14_W7.62mm, symbol Waveform:4013
Connections:
- new net AC_SQUARE: C3.2 (-), R3.1, RV2.1
- new net CLOCK_2K: TP1.1 (TP), U1.3 (OUT), U2.3 (CLK1)
- new net CTRL: C2.1, U1.5 (CTRL)
- new net DIGITAL_1K: C3.1 (+), U2.1 (Q1)
- new net DISCHARGE: R1.2, R2.1, U1.7 (DISCH)
- new net D_FEEDBACK: U2.2 (~Q1), U2.5 (D1)
- new net FREQ_R: C1.1, R2.2, RV1.1, RV1.2 (W), RV1.3, U1.2 (TRIG), U1.6 (THRES)
- new net GND: C1.2, C14.2, C15.2, C2.2, C20.2, C21.2, C26.2, C27.2, C28.2 (-), C29.1 (+), C30.2, C31.2, C32.2, C33.1, C34.2, C35.1, C36.2, C37.1, C38.2, C39.1, C40.2, C41.1, C42.2, C43.1, C44.2, C45.1, C46.2, C47.1, C48.2, C49.1, C50.2, C51.1, C52.2, C53.1, C54.2, C55.1, C56.2, C57.1, C58.2, C59.1, C8.2, C9.2, J5.2, J6.2, R3.2, RV12.3, RV13.2 (W), RV13.3, RV14.2 (W), RV14.3, RV17.3, RV18.2 (W), RV18.3, RV19.2 (W), RV19.3, RV2.3, RV22.3, RV3.2 (W), RV3.3, RV4.2 (W), RV4.3, RV7.3, RV8.2 (W), RV8.3, RV9.2 (W), RV9.3, TP18.1 (TP), U1.1 (GND), U10.3 (+), U10.5 (+), U12.3 (+), U13.3 (+), U13.5 (+), U15.3 (+), U16.3 (+), U16.5 (+), U2.11 (CLK2), U2.4 (RESET1), U2.6 (SET1), U2.7 (VSS), U2.8 (SET2), U2.9 (D2), U3.5 (+), U4.3 (+), U4.5 (+), U6.3 (+), U7.3 (+), U7.5 (+), U9.3 (+)
- new net H1_AMPLITUDE: R62.1, RV7.2 (W), TP6.1 (TP), U6.5 (+), U6.6 (-), U6.7 (OUT)
- new net H1_AP1: R13.1, R15.1, R17.1, U5.1 (OUT)
- new net H1_AP2: J1.1, R16.1, R18.1, TP5.1 (TP), U5.7 (OUT)
- new net H1_APINV1: R12.2, R13.2, U5.2 (-)
- new net H1_APINV2: R15.2, R16.2, U5.6 (-)
- new net H1_BPF1: C4.2, R8.1, R9.1, U4.1 (OUT)
- new net H1_BPF2: C6.2, R11.1, R12.1, R14.1, TP4.1 (TP), U4.7 (OUT)
- new net H1_INV1: C5.2, R8.2, U4.2 (-)
- new net H1_INV2: C7.2, R11.2, U4.6 (-)
- new net H1_LP1: C8.1, RV5.2 (W), RV5.3, U5.3 (+)
- new net H1_LP2: C9.1, RV6.2 (W), RV6.3, U5.5 (+)
- new net H1_NEG: J1.3, R19.1, U6.1 (OUT)
- new net H1_NODE1: C4.1, C5.1, R6.2, R7.1
- new net H1_NODE2: C6.1, C7.1, R10.1, R9.2
- new net H1_PHR1: R14.2, RV5.1
- new net H1_PHR2: R17.2, RV6.1
- new net H1_POLINV: R18.2, R19.2, U6.2 (-)
- new net H1_SELECT: J1.2, RV7.1
- new net H1_TUNE1: R7.2, RV3.1
- new net H1_TUNE2: R10.2, RV4.1
- new net H3_AMPLITUDE: R63.1, RV12.2 (W), TP9.1 (TP), U9.5 (+), U9.6 (-), U9.7 (OUT)
- new net H3_AP1: R27.1, R29.1, R31.1, U8.1 (OUT)
- new net H3_AP2: J2.1, R30.1, R32.1, TP8.1 (TP), U8.7 (OUT)
- new net H3_APINV1: R26.2, R27.2, U8.2 (-)
- new net H3_APINV2: R29.2, R30.2, U8.6 (-)
- new net H3_BPF1: C10.2, R22.1, R23.1, U7.1 (OUT)
- new net H3_BPF2: C12.2, R25.1, R26.1, R28.1, TP7.1 (TP), U7.7 (OUT)
- new net H3_INV1: C11.2, R22.2, U7.2 (-)
- new net H3_INV2: C13.2, R25.2, U7.6 (-)
- new net H3_LP1: C14.1, RV10.2 (W), RV10.3, U8.3 (+)
- new net H3_LP2: C15.1, RV11.2 (W), RV11.3, U8.5 (+)
- new net H3_NEG: J2.3, R33.1, U9.1 (OUT)
- new net H3_NODE1: C10.1, C11.1, R20.2, R21.1
- new net H3_NODE2: C12.1, C13.1, R23.2, R24.1
- new net H3_PHR1: R28.2, RV10.1
- new net H3_PHR2: R31.2, RV11.1
- new net H3_POLINV: R32.2, R33.2, U9.2 (-)
- new net H3_SELECT: J2.2, RV12.1
- new net H3_TUNE1: R21.2, RV8.1
- new net H3_TUNE2: R24.2, RV9.1
- new net H5_AMPLITUDE: R64.1, RV17.2 (W), TP12.1 (TP), U12.5 (+), U12.6 (-), U12.7 (OUT)
- new net H5_AP1: R41.1, R43.1, R45.1, U11.1 (OUT)
- new net H5_AP2: J3.1, R44.1, R46.1, TP11.1 (TP), U11.7 (OUT)
- new net H5_APINV1: R40.2, R41.2, U11.2 (-)
- new net H5_APINV2: R43.2, R44.2, U11.6 (-)
- new net H5_BPF1: C16.2, R36.1, R37.1, U10.1 (OUT)
- new net H5_BPF2: C18.2, R39.1, R40.1, R42.1, TP10.1 (TP), U10.7 (OUT)
- new net H5_INV1: C17.2, R36.2, U10.2 (-)
- new net H5_INV2: C19.2, R39.2, U10.6 (-)
- new net H5_LP1: C20.1, RV15.2 (W), RV15.3, U11.3 (+)
- new net H5_LP2: C21.1, RV16.2 (W), RV16.3, U11.5 (+)
- new net H5_NEG: J3.3, R47.1, U12.1 (OUT)
- new net H5_NODE1: C16.1, C17.1, R34.2, R35.1
- new net H5_NODE2: C18.1, C19.1, R37.2, R38.1
- new net H5_PHR1: R42.2, RV15.1
- new net H5_PHR2: R45.2, RV16.1
- new net H5_POLINV: R46.2, R47.2, U12.2 (-)
- new net H5_SELECT: J3.2, RV17.1
- new net H5_TUNE1: R35.2, RV13.1
- new net H5_TUNE2: R38.2, RV14.1
- new net H7_AMPLITUDE: R65.1, RV22.2 (W), TP15.1 (TP), U15.5 (+), U15.6 (-), U15.7 (OUT)
- new net H7_AP1: R55.1, R57.1, R59.1, U14.1 (OUT)
- new net H7_AP2: J4.1, R58.1, R60.1, TP14.1 (TP), U14.7 (OUT)
- new net H7_APINV1: R54.2, R55.2, U14.2 (-)
- new net H7_APINV2: R57.2, R58.2, U14.6 (-)
- new net H7_BPF1: C22.2, R50.1, R51.1, U13.1 (OUT)
- new net H7_BPF2: C24.2, R53.1, R54.1, R56.1, TP13.1 (TP), U13.7 (OUT)
- new net H7_INV1: C23.2, R50.2, U13.2 (-)
- new net H7_INV2: C25.2, R53.2, U13.6 (-)
- new net H7_LP1: C26.1, RV20.2 (W), RV20.3, U14.3 (+)
- new net H7_LP2: C27.1, RV21.2 (W), RV21.3, U14.5 (+)
- new net H7_NEG: J4.3, R61.1, U15.1 (OUT)
- new net H7_NODE1: C22.1, C23.1, R48.2, R49.1
- new net H7_NODE2: C24.1, C25.1, R51.2, R52.1
- new net H7_PHR1: R56.2, RV20.1
- new net H7_PHR2: R59.2, RV21.1
- new net H7_POLINV: R60.2, R61.2, U15.2 (-)
- new net H7_SELECT: J4.2, RV22.1
- new net H7_TUNE1: R49.2, RV18.1
- new net H7_TUNE2: R52.2, RV19.1
- new net OUT: J6.1, R69.2, TP17.1 (TP)
- new net RESTORE_INV: R67.2, R68.2, U16.6 (-)
- new net SOURCE_WIPER: RV2.2 (W), U3.3 (+)
- new net SQ: R20.1, R34.1, R4.1, R48.1, R6.1, TP2.1 (TP), U3.1 (OUT), U3.2 (-)
- new net SQ_INV: R5.1, TP3.1 (TP), U3.7 (OUT)
- new net SQ_INV_IN: R4.2, R5.2, U3.6 (-)
- new net SUM_INV: R62.2, R63.2, R64.2, R65.2, R66.2, U16.2 (-)
- new net SUM_NEG: R66.1, R67.1, U16.1 (OUT)
- new net SUM_RAW: R68.1, R69.1, TP16.1 (TP), U16.7 (OUT)
- new net VCC: C28.1 (+), C30.1, C31.1, C32.1, C34.1, C36.1, C38.1, C40.1, C42.1, C44.1, C46.1, C48.1, C50.1, C52.1, C54.1, C56.1, C58.1, J5.1, R1.1, U1.4 (RESET), U1.8 (VCC), U10.8 (V+), U11.8 (V+), U12.8 (V+), U13.8 (V+), U14.8 (V+), U15.8 (V+), U16.8 (V+), U2.10 (RESET2), U2.14 (VDD), U3.8 (V+), U4.8 (V+), U5.8 (V+), U6.8 (V+), U7.8 (V+), U8.8 (V+), U9.8 (V+)
- new net VEE: C29.2 (-), C33.2, C35.2, C37.2, C39.2, C41.2, C43.2, C45.2, C47.2, C49.2, C51.2, C53.2, C55.2, C57.2, C59.2, J5.3, U10.4 (V-), U11.4 (V-), U12.4 (V-), U13.4 (V-), U14.4 (V-), U15.4 (V-), U16.4 (V-), U3.4 (V-), U4.4 (V-), U5.4 (V-), U6.4 (V-), U7.4 (V-), U8.4 (V-), U9.4 (V-)
- no-connect marks 0 -> 2
Other:
- removed sheet harmonic_1
- removed sheet harmonic_3
- removed sheet harmonic_5
- removed sheet harmonic_7
- removed sheet power_sum
- removed sheet source
- note added: "1 kHz: TWO MFB BANDPASS SECTIONS -> TWO ALL-PASS SECTIONS -> POLARITY -> AMPLITUDE"
- note added: "3 kHz: TWO MFB BANDPASS SECTIONS -> TWO ALL-PASS SECTIONS -> POLARITY -> AMPLITUDE"
- note added: "5 kHz: TWO MFB BANDPASS SECTIONS -> TWO ALL-PASS SECTIONS -> POLARITY -> AMPLITUDE"
- note added: "7 kHz: TWO MFB BANDPASS SECTIONS -> TWO ALL-PASS SECTIONS -> POLARITY -> AMPLITUDE"
- note added: "ANALOG POWER AND LOCAL BYPASS: 100 nF at each supply pin"
- note added: "C29 positive terminal = GND"
- note added: "NE555 + TL082 FOURIER WAVEFORM SYNTHESIS — Rev B wired schematic"
- note added: "ONE shunt: default 2-3"
- note added: "REGULATED +/-12 V INPUT"
- note added: "Regulated +12 V / GND / -12 V. Signal wires are drawn explicitly. All labels are single-sheet local nets."
- note added: "SOURCE: 2 kHz clock / divide by two / DC blocking / 10 Vpp calibration"
- note added: "SUM AND OUTPUT"
- note removed: "NE555 2 kHz -> CD4013 /2 -> 10 Vpp SQ -> 1/3/5/7 kHz BPF -> phase / amplitude -> sum External regulated +12 V / GND / -12 V. High impedance output measurement."
- title: 1 kHz Fourier waveform synthesis -> Wired Fourier waveform synthesis
