File: hardware/waveform.sch (EAGLE design)
At the start: 190 parts, among them J1 PHASE_POLARITY, J2 PHASE_POLARITY, J3 PHASE_POLARITY, J4 PHASE_POLARITY, J5 POWER_12V, J6 WAVE_OUT, U1 NE555P, U10 TL082CP, U11 TL082CP, U12 TL082CP, U13 TL082CP, U14 TL082CP, U15 TL082CP, U16 TL082CP, U2 CD4013BE, U3 TL082CP, U4 TL082CP, U5 TL082CP, U6 TL082CP, U7 TL082CP, U8 TL082CP, U9 TL082CP

Commit message: Redraw waveform schematic as wired functional blocks for readable EDA import
Split TL082 amplifier and power units, replace the component grid with a single wired schematic and local net labels, and update both KiCad and EAGLE exchanges. Preserve all PCB copper and pad geometry; verify 491 pin connections, zero ERC/DRC issues, and EAGLE PCB round-trip checks. Add clearly named RevB wired download packages.
Connections:
- net GND: now also U10A.3, U10B.5, U12A.3, U13A.3, U13B.5, U15A.3, U16A.3, U16B.5, U3B.5, U4A.3, U4B.5, U6A.3, U7A.3, U7B.5, U9A.3; no longer U10.3, U10.5, U12.3, U13.3, U13.5, U15.3, U16.3, U16.5, U3.5, U4.3, U4.5, U6.3, U7.3, U7.5, U9.3
- net H1_AMPLITUDE: now also U6B.5; no longer U6.5
- net H1_AP1: now also U5A.1; no longer U5.1
- net H1_AP2: now also U5B.7; no longer U5.7
- net H1_APINV1: now also U5A.2; no longer U5.2
- net H1_APINV2: now also U5B.6; no longer U5.6
- net H1_BPF1: now also U4A.1; no longer U4.1
- net H1_BPF2: now also U4B.7; no longer U4.7
- net H1_INV1: now also U4A.2; no longer U4.2
- net H1_INV2: now also U4B.6; no longer U4.6
- net H1_LP1: now also U5A.3; no longer U5.3
- net H1_LP2: now also U5B.5; no longer U5.5
- net H1_NEG: now also U6A.1; no longer U6.1
- net H1_OUT: now also U6B.6, U6B.7; no longer U6.6, U6.7
- net H1_POLINV: now also U6A.2; no longer U6.2
- net H3_AMPLITUDE: now also U9B.5; no longer U9.5
- net H3_AP1: now also U8A.1; no longer U8.1
- net H3_AP2: now also U8B.7; no longer U8.7
- net H3_APINV1: now also U8A.2; no longer U8.2
- net H3_APINV2: now also U8B.6; no longer U8.6
- net H3_BPF1: now also U7A.1; no longer U7.1
- net H3_BPF2: now also U7B.7; no longer U7.7
- net H3_INV1: now also U7A.2; no longer U7.2
- net H3_INV2: now also U7B.6; no longer U7.6
- net H3_LP1: now also U8A.3; no longer U8.3
- net H3_LP2: now also U8B.5; no longer U8.5
- net H3_NEG: now also U9A.1; no longer U9.1
- net H3_OUT: now also U9B.6, U9B.7; no longer U9.6, U9.7
- net H3_POLINV: now also U9A.2; no longer U9.2
- net H5_AMPLITUDE: now also U12B.5; no longer U12.5
- net H5_AP1: now also U11A.1; no longer U11.1
- net H5_AP2: now also U11B.7; no longer U11.7
- net H5_APINV1: now also U11A.2; no longer U11.2
- net H5_APINV2: now also U11B.6; no longer U11.6
- net H5_BPF1: now also U10A.1; no longer U10.1
- net H5_BPF2: now also U10B.7; no longer U10.7
- net H5_INV1: now also U10A.2; no longer U10.2
- net H5_INV2: now also U10B.6; no longer U10.6
- net H5_LP1: now also U11A.3; no longer U11.3
- net H5_LP2: now also U11B.5; no longer U11.5
- net H5_NEG: now also U12A.1; no longer U12.1
- net H5_OUT: now also U12B.6, U12B.7; no longer U12.6, U12.7
- net H5_POLINV: now also U12A.2; no longer U12.2
- net H7_AMPLITUDE: now also U15B.5; no longer U15.5
- net H7_AP1: now also U14A.1; no longer U14.1
- net H7_AP2: now also U14B.7; no longer U14.7
- net H7_APINV1: now also U14A.2; no longer U14.2
- net H7_APINV2: now also U14B.6; no longer U14.6
- net H7_BPF1: now also U13A.1; no longer U13.1
- net H7_BPF2: now also U13B.7; no longer U13.7
- net H7_INV1: now also U13A.2; no longer U13.2
- net H7_INV2: now also U13B.6; no longer U13.6
- net H7_LP1: now also U14A.3; no longer U14.3
- net H7_LP2: now also U14B.5; no longer U14.5
- net H7_NEG: now also U15A.1; no longer U15.1
- net H7_OUT: now also U15B.6, U15B.7; no longer U15.6, U15.7
- net H7_POLINV: now also U15A.2; no longer U15.2
- net RESTORE_INV: now also U16B.6; no longer U16.6
- net SOURCE_WIPER: now also U3A.3; no longer U3.3
- net SQ: now also U3A.1, U3A.2; no longer U3.1, U3.2
- net SQ_INV: now also U3B.7; no longer U3.7
- net SQ_INV_IN: now also U3B.6; no longer U3.6
- net SUM_INV: now also U16A.2; no longer U16.2
- net SUM_NEG: now also U16A.1; no longer U16.1
- net SUM_RAW: now also U16B.7; no longer U16.7
- net VCC: now also U10P.8, U11P.8, U12P.8, U13P.8, U14P.8, U15P.8, U16P.8, U3P.8, U4P.8, U5P.8, U6P.8, U7P.8, U8P.8, U9P.8; no longer U10.8, U11.8, U12.8, U13.8, U14.8, U15.8, U16.8, U3.8, U4.8, U5.8, U6.8, U7.8, U8.8, U9.8
- net VEE: now also U10P.4, U11P.4, U12P.4, U13P.4, U14P.4, U15P.4, U16P.4, U3P.4, U4P.4, U5P.4, U6P.4, U7P.4, U8P.4, U9P.4; no longer U10.4, U11.4, U12.4, U13.4, U14.4, U15.4, U16.4, U3.4, U4.4, U5.4, U6.4, U7.4, U8.4, U9.4
Other:
- note added: "1 kHz: TWO MFB BANDPASS SECTIONS -> TWO ALL-PASS SECTIONS -> POLARITY -> AMPLITUDE"
- note added: "3 kHz: TWO MFB BANDPASS SECTIONS -> TWO ALL-PASS SECTIONS -> POLARITY -> AMPLITUDE"
- note added: "5 kHz: TWO MFB BANDPASS SECTIONS -> TWO ALL-PASS SECTIONS -> POLARITY -> AMPLITUDE"
- note added: "7 kHz: TWO MFB BANDPASS SECTIONS -> TWO ALL-PASS SECTIONS -> POLARITY -> AMPLITUDE"
- note added: "ANALOG POWER AND LOCAL BYPASS: 100 nF at each supply pin"
- note added: "C29 positive terminal = GND"
- note added: "NE555 + TL082 FOURIER WAVEFORM SYNTHESIS — Rev B wired schematic"
- note added: "ONE shunt: default 2-3"
- note added: "REGULATED +/-12 V INPUT"
- note added: "Regulated +12 V / GND / -12 V. Signal wires are drawn explicitly. All labels are single-sheet local nets."
- note added: "SOURCE: 2 kHz clock / divide by two / DC blocking / 10 Vpp calibration"
- note added: "SUM AND OUTPUT"
- note removed: "Waveform synthesis: harmonic_1 (VCC=+12V, VEE=-12V)"
- note removed: "Waveform synthesis: harmonic_3 (VCC=+12V, VEE=-12V)"
- note removed: "Waveform synthesis: harmonic_5 (VCC=+12V, VEE=-12V)"
- note removed: "Waveform synthesis: harmonic_7 (VCC=+12V, VEE=-12V)"
- note removed: "Waveform synthesis: power_sum (VCC=+12V, VEE=-12V)"
- note removed: "Waveform synthesis: source (VCC=+12V, VEE=-12V)"
